File: KiCAD/me310-diff-amp/me310-diff-amp.kicad_sch (KiCad schematic)
At the start: 24 parts, among them U1 LM741, U2 LM741

Commit message: BOM
Parts:
- added N1, N2: DIP-8 Socket, symbol Mechanical:Housing
- C1, C2, C3, C4: value C -> 0.1uF; CatNo (none) -> 399-4264-ND; Vendor (none) -> DigiKey
- R1, R3, R4, R5, R6: value R_US -> 10k; CatNo (none) -> CF14JT10K0CT-ND; Vendor (none) -> DigiKey
- R2: value R_US -> 100k; CatNo (none) -> CF14JT91K0CT-ND; Vendor (none) -> DigiKey
- U1, U2: CatNo (none) -> 24539; Vendor (none) -> Jameco?

Commit message: as built V1
Parts:
- R1, R3, R5: value 10k -> 100k; CatNo CF14JT10K0CT-ND -> CF14JT100KCT-ND
- R2: value 100k -> 1M; CatNo CF14JT91K0CT-ND -> CF14JT1M00CT-ND
- R4, R6: value 10k -> 1M; CatNo CF14JT10K0CT-ND -> CF14JT1M00CT-ND
- U1, U2: CatNo 24539 -> LM741CNNS/NOPB-ND; Vendor Jameco? -> DigiKey
Changed lines of the file:
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@@
 (kicad_sch (version 20230121) (generator eeschema)
-  (paper "A4")
+  (paper "USLetter")
   (junction (at 110.49 96.52) (diameter 0) (color 0 0 0 0)
   )
@@
       (effects (font (size 1.27 1.27)))
     )
-    (property "Value" "10k" (at 146.05 77.47 90)
+    (property "Value" "100k" (at 146.05 77.47 90)
       (effects (font (size 1.27 1.27)))
     )
@@
       (effects (font (size 1.27 1.27)) hide)
     )
-    (property "CatNo" "CF14JT10K0CT-ND" (at 142.24 80.01 0)
+    (property "CatNo" "CF14JT100KCT-ND" (at 142.24 80.01 0)
       (effects (font (size 1.27 1.27)) hide)
     )
@@
       (effects (font (size 1.27 1.27)))
     )
-    (property "Value" "10k" (at 168.91 99.06 90)
+    (property "Value" "1M" (at 168.91 99.06 90)
       (effects (font (size 1.27 1.27)))
     )
@@
       (effects (font (size 1.27 1.27)) hide)
     )
-    (property "CatNo" "CF14JT10K0CT-ND" (at 165.1 96.52 0)
+    (property "CatNo" "CF14JT1M00CT-ND" (at 165.1 96.52 0)
       (effects (font (size 1.27 1.27)) hide)
     )
@@
       (effects (font (size 1.27 1.27)) hide)
     )
-    (property "CatNo" "24539" (at 165.1 80.01 0)
-      (effects (font (size 1.27 1.27)) hide)
-    )
-    (property "Vendor" "Jameco?" (at 165.1 80.01 0)
+    (property "CatNo" "LM741CNNS/NOPB-ND" (at 165.1 80.01 0)
+      (effects (font (size 1.27 1.27)) hide)
+    )
+    (property "Vendor" "DigiKey" (at 165.1 80.01 0)
       (effects (font (size 1.27 1.27)) hide)
     )
@@
       (effects (font (size 1.27 1.27)))
     )
-    (property "Value" "100k" (at 128.27 93.98 90)
+    (property "Value" "1M" (at 128.27 93.98 90)
       (effects (font (size 1.27 1.27)))
     )
@@
       (effects (font (size 1.27 1.27)) hide)
     )
-    (property "CatNo" "CF14JT91K0CT-ND" (at 124.46 96.52 0)
+    (property "CatNo" "CF14JT1M00CT-ND" (at 124.46 96.52 0)
       (effects (font (size 1.27 1.27)) hide)
     )
@@
       (effects (font (size 1.27 1.27)))
     )
-    (property "Value" "10k" (at 102.87 85.09 0)
+    (property "Value" "1M" (at 102.87 85.09 0)
       (effects (font (size 1.27 1.27)))
     )
@@
       (effects (font (size 1.27 1.27)) hide)
     )
-    (property "CatNo" "CF14JT10K0CT-ND" (at 106.68 83.82 0)
+    (property "CatNo" "CF14JT1M00CT-ND" (at 106.68 83.82 0)
       (effects (font (size 1.27 1.27)) hide)
     )
@@
       (effects (font (size 1.27 1.27)))
     )
-    (property "Value" "10k" (at 105.41 74.93 90)
+    (property "Value" "100k" (at 105.41 74.93 90)
       (effects (font (size 1.27 1.27)))
     )
@@
       (effects (font (size 1.27 1.27)) hide)
     )
-    (property "CatNo" "CF14JT10K0CT-ND" (at 101.6 77.47 0)
+    (property "CatNo" "CF14JT100KCT-ND" (at 101.6 77.47 0)
       (effects (font (size 1.27 1.27)) hide)
     )
@@
       (effects (font (size 1.27 1.27)))
     )
-    (property "Value" "10k" (at 105.41 93.98 90)
+    (property "Value" "100k" (at 105.41 93.98 90)
       (effects (font (size 1.27 1.27)))
     )
@@
       (effects (font (size 1.27 1.27)) hide)
     )
-    (property "CatNo" "CF14JT10K0CT-ND" (at 101.6 96.52 0)
+    (property "CatNo" "CF14JT100KCT-ND" (at 101.6 96.52 0)
       (effects (font (size 1.27 1.27)) hide)
     )
@@
       (effects (font (size 1.27 1.27)) hide)
     )
-    (property "CatNo" "24539" (at 119.38 80.01 0)
-      (effects (font (size 1.27 1.27)) hide)
-    )
-    (property "Vendor" "Jameco?" (at 119.38 80.01 0)
-      (effects (font (size 1.27 1.27)) hide)
-    )
+    (property "CatNo" "LM741CNNS/NOPB-ND" (at 119.38 80.01 0)
+      (effects (font (size 1.27 1.27)) hide)
+    )
+    (property "Vendor" "DigiKey" (at 119.38 80.01 0)
+      (effects (font (size 1.27 1.27)) hide)
+    )
