File: KiCAD/me310-diff-amp/me310-diff-amp.kicad_pcb (KiCad board)
At the start: 2 copper layers, 63.5 x 63.5 mm, 24 parts, among them U1 LM741, U2 LM741

Commit message: Rev 2.0 ready?
Parts:
- moved C2 80.4 mm to (153.7, 94.6), turned to 180 degrees
- moved C4 71.0 mm to (146.1, 111.8)
- moved R5 15.9 mm to (138.4, 108.0), turned to 90 degrees
- moved R1 11.5 mm to (108.6, 110.5)
- moved C1 11.4 mm to (133.3, 95.2), turned to 180 degrees
- moved R4 9.09 mm to (108.6, 102.9)
- moved C3 8.93 mm to (125.8, 111.8), turned to 0 degrees
- moved U2 6.35 mm to (146.1, 99.7)
- moved U1 6.29 mm to (125.7, 99.7)
- moved R3 5.39 mm to (108.6, 95.2)
- moved TP4 4.58 mm to (104.1, 95.2)
- moved TP5 4.58 mm to (104.1, 110.5)
- moved TP6 4.58 mm to (104.1, 102.9)
- moved R2 3.81 mm to (123.8, 117.5)
- moved R6 3.81 mm to (154.9, 117.5)
Routing:
- net -15V: track 0.00 -> 85.4 mm, vias 0 -> 2
- net +15V: track 0.00 -> 64.8 mm
- net Net-(U1--): track 0.00 -> 37.1 mm
- net Net-(U2--): track 0.00 -> 31.5 mm
- net Net-(R6-Pad1): track 0.00 -> 22.8 mm
- net Net-(R2-Pad2): track 0.00 -> 17.7 mm
- net Net-(U1-+): track 0.00 -> 15.4 mm
- net Net-(R3-Pad1): track 0.00 -> 4.44 mm
- added copper zone on B.Cu, net GND
Other:
- board text added: "+15V"
- board text added: "-15V"
- board text added: "Inverting Differential Amplifier V2.0 - E. Hazen - 2024-02"
- board text added: "ME310"

Commit message: Rev 2.1 changes, README
Routing:
- net Net-(R1-Pad1): track 0.00 -> 4.44 mm
Other:
- board text added: "Inverting Differential Amplifier V2.1 - E. Hazen - 2024-04"
- board text removed: "Inverting Differential Amplifier V2.0 - E. Hazen - 2024-02"
