File: KiCAD/girl_scouts_blinker/girl_scouts_blinker.kicad_sch (KiCad schematic)
At the start: 16 parts, among them SW1 SW_Push, SW2 SW_Push, SW3 SW_SPST, U1 ATtiny85-20P

Commit message: add programming connector and RST R
Parts:
- added J1: AVR-ISP-6, Connector_PinHeader_2.54mm:PinHeader_2x03_P2.54mm_Vertical, symbol Connector:AVR-ISP-6
- added N1: IC Socket, symbol Mechanical:Housing
- added R1: 10k, Resistor_THT:R_Axial_DIN0207_L6.3mm_D2.5mm_P10.16mm_Horizontal, symbol Device:R_US
- C1, C2: CatNo (none) -> 445-173588-1-ND; MfgNo (none) -> FG28X7R1H104KNT06
- D1, D3, D4: value NeoPixel_THT -> Adafruit NeoPixel_THT; CatNo (none) -> 1938
- D2: CatNo (none) -> 4878-1N4002CT-ND; MfgNo (none) -> 1N4002
- FID1: now not fitted
- SW1, SW2: MfgNo (none) -> CFM14JT10K0
- SW3: footprint my_slide_sw:sw_spdt_p4.8mm -> my_slide_sw:Slide_SLW-1711575-5A-N-D; CatNo (none) -> 2223-SLW-1711575-5A-N-D-ND; MfgNo (none) -> SLW-1711575-5A-N-D
- U1: CatNo (none) -> ATTINY85-20PU-ND; MfgNo (none) -> ATTINY85-20PU
Connections:
- net +5V: now also J1.2 (VCC), R1.1
- net GND: now also J1.6 (GND)
- net MISO: now also J1.1 (MISO)
- net MOSI: now also J1.4 (MOSI)
- net SCK: now also J1.3 (SCK)
- net nRST: now reaches U1.1 (~{RESET}/PB5)
- net nRST: now also J1.5 (~{RST}), R1.2
Other:
- note added: "Boston University EPIC"
- note added: "LED multi-color blinker Soldering project"

Commit message: layout v1.1 done?
Parts:
- removed BT1: Battery, Connector_PinHeader_2.54mm:PinHeader_1x02_P2.54mm_Vertical, symbol Device:Battery
- removed D2: 1N4002, Diode_THT:D_DO-41_SOD81_P10.16mm_Horizontal, symbol Diode:1N4002
- added B1: BC9VPC, my_footprints:BC9VPC_MPD, symbol PC9VPC:BC9VPC
- added U2: LM7805_TO220, Package_TO_SOT_THT:TO-220-3_Horizontal_TabDown, symbol Regulator_Linear:LM7805_TO220
- SW1, SW2: footprint push_sw:BTN-B3F-1000 -> my_cherry:SW_Cherry_MX_1.00u_PCB
Connections:
- net +5V: now also U2.3 (VO)
- net +6V: now also B1.1
- net GND: now also B1.2, U2.2 (GND)
- net at SW3.2 (B): now also U2.1 (VI)

Commit message: ready to order?
Parts:
- B1: CatNo (none) -> BC9VPC-ND; MfgNo (none) -> BC9VPC
- H1, H2, H3, H4: now not fitted
- U2: CatNo (none) -> 497-1443-5-ND; MfgNo (none) -> L7805CV
